Commit message: chore: align robot_vog package rules
Migrate the package to ament_cmake_python, update launch/config organization, add package tests and align lint configuration with the agreed ROS 2 package rules.

File: urdf/includes/fork_simple_module.xacro (robot description, xacro)
@@ -1,11 +1,8 @@
 <?xml version="1.0"?>
-<robot name="fork_module" xmlns:xacro="http://www.ros.org/wiki/xacro" xmlns:gz="http://gazebosim.org/schema">
-  <!---->
-  <!--
-  Be aware that if a property is not defined in this it is defined in the included model above.
-  -->
-  <xacro:include filename="${robotics_description_pkg_dir}/urdf/sensors/all_sensors_macro.xacro"/>
-  <xacro:include filename="${robotics_description_pkg_dir}/urdf/extras/fork_simple/fork_simple_macro.xacro"/>
-  <xacro:include filename="${robotics_description_pkg_dir}/urdf/extras/fork_simple/generic_macros/plugin_fork_joint_f64_pos_pid_macro.xacro"/>
+<robot name="robot_vog_forklift_module" xmlns:xacro="http://www.ros.org/wiki/xacro">
+  <!-- This module extends the common VOG platform with the forklift and its sensor layout. -->
+  <xacro:include filename="$(find robotics_description)/urdf/sensors/all_sensors_macro.xacro"/>
+  <xacro:include filename="$(find robotics_description)/urdf/extras/fork_simple/fork_simple_macro.xacro"/>
+  <xacro:include filename="$(find robotics_description)/urdf/extras/fork_simple/generic_macros/plugin_fork_joint_f64_pos_pid_macro.xacro"/>
   <!-- ===================================================================== -->
   <!-- ARGS -->
@@ -114,8 +111,4 @@
   <xacro:property name="fork_carriage_mount_y" value="0"/>
   <xacro:property name="fork_carriage_mount_z" value="${-ground_clearance + fork_rest_clearance}"/>
-  <xacro:property name="tine_size_x"           value="1.20"/>
-  <xacro:property name="tine_size_y"           value="0.12"/>
-  <xacro:property name="tine_size_z"           value="0.06"/>
-  <xacro:property name="tine_separation"       value="0.25"/>
   <xacro:fork_simple name="${fork_name}"
                      prefix="${robot_prefix}"
@@ -173,5 +166,5 @@
   The frame of the mesh is located at its center.
   Sizes of the mesh are: (size_x = 0.025053 m, size_y = 0.089909 m, size_z = 0.025000 m)
-  The frame of the mesh is located, w.r.t ${prefix}${name}_bottom_screw_frame, at
+  The mesh frame is located relative to ${prefix}${name}_bottom_screw_frame at
   (x = 0.002375 m, y = 0 m, z = 0.0125 m, R = 0 rad, P = 0 rad, Y = 0 rad).
   The bottom face of the mesh is touching the root frame of the camera.
@@ -194,6 +187,6 @@
                              use_c_mesh="${fork_rgbd_use_c_mesh}"
                              joint_parent_fr_root_fr="${fork_rgbd_mount_x} ${fork_rgbd_mount_y} ${fork_rgbd_mount_z} 0 0 0"
-                             use_sensor_frames_and_joints="${use_sim_mode}"
-                             sim_rgbd_enabled="${use_sim_mode and fork_camera_rgbd_sim_enabled}"
+                             use_sensor_frames_and_joints="True"
+                             sim_rgbd_enabled="${fork_camera_rgbd_sim_enabled}"
                              sim_rgbd_use_gravity="${fork_camera_rgbd_sim_use_gravity}"
                              sim_rgbd_always_on="${fork_camera_rgbd_sim_always_on}"
@@ -215,5 +208,5 @@
                              sim_rgbd_distortion_center="${fork_camera_rgbd_sim_distortion_center}"
                              sim_rgbd_gaussian_noise="${fork_camera_rgbd_sim_gaussian_noise}"
-                             sim_infra1_enabled="${use_sim_mode and fork_camera_infra1_sim_enabled}"
+                             sim_infra1_enabled="${fork_camera_infra1_sim_enabled}"
                              sim_infra1_use_gravity="${fork_camera_infra1_sim_use_gravity}"
                              sim_infra1_always_on="${fork_camera_infra1_sim_always_on}"
@@ -234,5 +227,5 @@
                              sim_infra1_distortion_center="${fork_camera_infra1_sim_distortion_center}"
                              sim_infra1_gaussian_noise="${fork_camera_infra1_sim_gaussian_noise}"
-                             sim_infra2_enabled="${use_sim_mode and fork_camera_infra2_sim_enabled}"
+                             sim_infra2_enabled="${fork_camera_infra2_sim_enabled}"
                              sim_infra2_use_gravity="${fork_camera_infra2_sim_use_gravity}"
                              sim_infra2_always_on="${fork_camera_infra2_sim_always_on}"
@@ -315,5 +308,5 @@
       c_mesh_use_low_res="${front_top_lidar_c_mesh_use_low_res}"
       joint_parent_fr_root_fr="${front_top_lidar_joint_parent_fr_root_fr}"
-      sim_lidar_enabled="${use_sim_mode and front_top_lidar_sim_enabled}"
+      sim_lidar_enabled="${front_top_lidar_sim_enabled}"
       sim_lidar_always_on="${front_top_lidar_sim_always_on}"
       sim_lidar_visualize="${front_top_lidar_sim_visualize}"
@@ -325,5 +318,5 @@
       sim_lidar_dist_span="${front_top_lidar_sim_dist_span}"
       sim_lidar_gaussian_noise="${front_top_lidar_sim_gaussian_noise}"
-      sim_imu_enabled="${use_sim_mode and front_top_lidar_imu_sim_enabled}"
+      sim_imu_enabled="${front_top_lidar_imu_sim_enabled}"
       sim_imu_use_gravity="${front_top_lidar_imu_sim_use_gravity}"
       sim_imu_always_on="${front_top_lidar_imu_sim_always_on}"
@@ -376,14 +369,14 @@
     c_mesh_use_low_res="${front_bottom_lidar_c_mesh_use_low_res}"
     joint_parent_fr_root_fr="${front_bottom_lidar_joint_parent_fr_root_fr}"
-    sim_lidar_enabled="${use_sim_mode and front_bottom_lidar_sim_enabled}"
-    sim_lidar_always_on="${front_bottom_lidar_sim_always_on}"
-    sim_lidar_visualize="${front_bottom_lidar_sim_visualize}"
-    sim_lidar_update_rate="${front_bottom_lidar_sim_update_rate}"
-    sim_lidar_hor_fov_deg="${front_bottom_lidar_sim_hor_fov_deg}"
-    sim_lidar_hor_res_deg="${front_bottom_lidar_sim_hor_res_deg}"
-    sim_lidar_dist_span="${front_bottom_lidar_sim_dist_span}"
-    sim_lidar_gaussian_noise="${front_bottom_lidar_sim_gaussian_noise}"
+    sim_enabled="${front_bottom_lidar_sim_enabled}"
+    sim_always_on="${front_bottom_lidar_sim_always_on}"
+    sim_visualize="${front_bottom_lidar_sim_visualize}"
+    sim_update_rate="${front_bottom_lidar_sim_update_rate}"
+    sim_hor_fov_deg="${front_bottom_lidar_sim_hor_fov_deg}"
+    sim_hor_res_deg="${front_bottom_lidar_sim_hor_res_deg}"
+    sim_dist_span="${front_bottom_lidar_sim_dist_span}"
+    sim_gaussian_noise="${front_bottom_lidar_sim_gaussian_noise}"
     namespace="${robot_namespace}"
-    sim_lidar_topic="${front_bottom_lidar_sim_topic}"/>
+    sim_topic="${front_bottom_lidar_sim_topic}"/>
   <!-- ===================================================================== -->
   <!-- BACK TOP ROBOSENSE AIRY -->
@@ -440,5 +433,5 @@
       c_mesh_use_low_res="${back_top_lidar_c_mesh_use_low_res}"
       joint_parent_fr_root_fr="${back_top_lidar_joint_parent_fr_root_fr}"
-      sim_lidar_enabled="${use_sim_mode and back_top_lidar_sim_enabled}"
+      sim_lidar_enabled="${back_top_lidar_sim_enabled}"
       sim_lidar_always_on="${back_top_lidar_sim_always_on}"
       sim_lidar_visualize="${back_top_lidar_sim_visualize}"
@@ -450,5 +443,5 @@
       sim_lidar_dist_span="${back_top_lidar_sim_dist_span}"
       sim_lidar_gaussian_noise="${back_top_lidar_sim_gaussian_noise}"
-      sim_imu_enabled="${use_sim_mode and back_top_lidar_imu_sim_enabled}"
+      sim_imu_enabled="${back_top_lidar_imu_sim_enabled}"
       sim_imu_use_gravity="${back_top_lidar_imu_sim_use_gravity}"
       sim_imu_always_on="${back_top_lidar_imu_sim_always_on}"
@@ -464,5 +457,5 @@
       sim_lidar_base_topic="${back_top_lidar_sim_base_topic}"
       sim_imu_topic="${back_top_lidar_imu_sim_topic}"/>
-  <xacro:if value="${use_sim_mode}">
+  <xacro:if value="${sim_file != ''}">
     <gazebo>
       <!--
@@ -476,4 +469,7 @@
       <xacro:if value="${fork_controller_sim_cfg.get('enabled', False)}">
         <xacro:property name="fork_topic" value="${fork_controller_sim_cfg.get('topic', '')}"/>
+        <xacro:if value="${fork_topic == ''}">
+          ${xacro.fatal("fork_controller.topic is required when fork_controller.enabled is true.")}
+        </xacro:if>
         <xacro:if value="${fork_topic != ''}">
           <xacro:plugin_fork_joint_f64_pos_pid

File: urdf/models/model_base.xacro (robot description, xacro)
@@ -1,4 +1,4 @@
 <?xml version="1.0"?>
-<robot name="vog_base" xmlns:xacro="http://www.ros.org/wiki/xacro" xmlns:gz="http://gazebosim.org/schema">
+<robot name="vog_base" xmlns:xacro="http://www.ros.org/wiki/xacro">
   <!--
   This file publishes the `base` model of the `robot_vog` family.
@@ -6,8 +6,6 @@
   -->
   <xacro:include filename="$(find robot_vog)/urdf/includes/common.xacro"/>
-  <!--
-  Be aware that if a property is not defined in this it is defined in the included model above.
-  -->
-  <xacro:if value="${use_sim_mode}">
+  <!-- A non-empty sim_file adds the simulation-only joint-state publisher. -->
+  <xacro:if value="${sim_file != ''}">
     <gazebo>
       <!--
@@ -19,5 +17,8 @@
         <xacro:property name="js_topic"
                         value="${joint_state_publisher_sim_cfg.get('topic', '')}"/>
-        <!-- No topic, no Gazebo plugin -->
+        <xacro:if value="${js_topic == ''}">
+          ${xacro.fatal(
+            "joint_state_publisher.topic is required when joint_state_publisher.enabled is true.")}
+        </xacro:if>
         <xacro:if value="${js_topic != ''}">
           <xacro:resolve_topic prop_id="resolved_js_topic"
@@ -26,12 +27,12 @@
           <xacro:plugin_joint_state_publisher topic="${resolved_js_topic}">
             <joint_names>
-              <joint_name>${robot_prefix}${steerable_wheel_0_name}_steering_joint</joint_name>
-              <joint_name>${robot_prefix}${steerable_wheel_0_name}_rotation_joint</joint_name>
-              <joint_name>${robot_prefix}${steerable_wheel_1_name}_steering_joint</joint_name>
-              <joint_name>${robot_prefix}${steerable_wheel_1_name}_rotation_joint</joint_name>
-              <joint_name>${robot_prefix}${steerable_wheel_2_name}_steering_joint</joint_name>
-              <joint_name>${robot_prefix}${steerable_wheel_2_name}_rotation_joint</joint_name>
-              <joint_name>${robot_prefix}${steerable_wheel_3_name}_steering_joint</joint_name>
-              <joint_name>${robot_prefix}${steerable_wheel_3_name}_rotation_joint</joint_name>
+              <joint_name>${robot_prefix}${front_left_wheel_name}_steering_joint</joint_name>
+              <joint_name>${robot_prefix}${front_left_wheel_name}_rotation_joint</joint_name>
+              <joint_name>${robot_prefix}${front_right_wheel_name}_steering_joint</joint_name>
+              <joint_name>${robot_prefix}${front_right_wheel_name}_rotation_joint</joint_name>
+              <joint_name>${robot_prefix}${rear_left_wheel_name}_steering_joint</joint_name>
+              <joint_name>${robot_prefix}${rear_left_wheel_name}_rotation_joint</joint_name>
+              <joint_name>${robot_prefix}${rear_right_wheel_name}_steering_joint</joint_name>
+              <joint_name>${robot_prefix}${rear_right_wheel_name}_rotation_joint</joint_name>
             </joint_names>
           </xacro:plugin_joint_state_publisher>

File: urdf/models/model_forklift.xacro (robot description, xacro)
@@ -3,8 +3,7 @@
   This file publishes the `forklift` model of the `robot_vog` family.
   The robot name inside the URDF stays `vog_forklift`.
-  The model is a VOG robot with 4 steerable wheels that includes the
-  fork_simple module.
-  The fork_simple module contains:
-  - A simlpe fork.
+  This model extends the common VOG platform with the forklift module.
+  The forklift module contains:
+  - A simple fork.
   - A realsense d435 camera (rgbd) mounted on the fork.
   - A Robosense Airy lidar mounted on the back of the robot.
@@ -12,5 +11,5 @@
   - A front bottom lidar mounted on the robot body.
 -->
-<robot name="vog_forklift" xmlns:xacro="http://www.ros.org/wiki/xacro" xmlns:gz="http://gazebosim.org/schema">
+<robot name="vog_forklift" xmlns:xacro="http://www.ros.org/wiki/xacro">
   <!-- ===================================================================== -->
   <!-- INCLUDES -->
@@ -22,5 +21,5 @@
   This model file only adds the Gazebo joint state publisher for the full assembled robot.
   -->
-  <xacro:if value="${use_sim_mode}">
+  <xacro:if value="${sim_file != ''}">
     <gazebo>
       <xacro:property name="joint_state_publisher_sim_cfg"
@@ -28,4 +27,8 @@
       <xacro:if value="${joint_state_publisher_sim_cfg.get('enabled', False)}">
         <xacro:property name="js_topic" value="${joint_state_publisher_sim_cfg.get('topic', '')}"/>
+        <xacro:if value="${js_topic == ''}">
+          ${xacro.fatal(
+            "joint_state_publisher.topic is required when joint_state_publisher.enabled is true.")}
+        </xacro:if>
         <xacro:if value="${js_topic != ''}">
           <xacro:resolve_topic prop_id="resolved_js_topic"
@@ -35,12 +38,12 @@
             <joint_names>
               <joint_name>${robot_prefix}${fork_name}_carriage_joint</joint_name>
-              <joint_name>${robot_prefix}${steerable_wheel_0_name}_steering_joint</joint_name>
-              <joint_name>${robot_prefix}${steerable_wheel_0_name}_rotation_joint</joint_name>
-              <joint_name>${robot_prefix}${steerable_wheel_1_name}_steering_joint</joint_name>
-              <joint_name>${robot_prefix}${steerable_wheel_1_name}_rotation_joint</joint_name>
-              <joint_name>${robot_prefix}${steerable_wheel_2_name}_steering_joint</joint_name>
-              <joint_name>${robot_prefix}${steerable_wheel_2_name}_rotation_joint</joint_name>
-              <joint_name>${robot_prefix}${steerable_wheel_3_name}_steering_joint</joint_name>
-              <joint_name>${robot_prefix}${steerable_wheel_3_name}_rotation_joint</joint_name>
+              <joint_name>${robot_prefix}${front_left_wheel_name}_steering_joint</joint_name>
+              <joint_name>${robot_prefix}${front_left_wheel_name}_rotation_joint</joint_name>
+              <joint_name>${robot_prefix}${front_right_wheel_name}_steering_joint</joint_name>
+              <joint_name>${robot_prefix}${front_right_wheel_name}_rotation_joint</joint_name>
+              <joint_name>${robot_prefix}${rear_left_wheel_name}_steering_joint</joint_name>
+              <joint_name>${robot_prefix}${rear_left_wheel_name}_rotation_joint</joint_name>
+              <joint_name>${robot_prefix}${rear_right_wheel_name}_steering_joint</joint_name>
+              <joint_name>${robot_prefix}${rear_right_wheel_name}_rotation_joint</joint_name>
             </joint_names>
           </xacro:plugin_joint_state_publisher>
