Commit message: refactor: split rbvogui common package
Rename the package identity to robot_rbvogui_common and keep only shared base resources in this repository.

Remove forklift-specific configuration, launches, scripts, and dependencies so they can live in the forklift package.

File: urdf/common.xacro (robot description, xacro)
@@ -1,6 +1,6 @@
 <?xml version="1.0"?>
-<robot name="robot_vog_common" xmlns:xacro="http://www.ros.org/wiki/xacro">
-  <!--
-  Common xacro file for the VOG robot with 4 steerable wheels.
+<robot name="rbvogui_common" xmlns:xacro="http://www.ros.org/wiki/xacro">
+  <!--
+  Common xacro file for the RB-VOGUI robot with 4 steerable wheels.
   THIS FILE IS NOT A COMPLETE ROBOT MODEL, IT IS MEANT TO BE INCLUDED IN THE SPECIFIC ROBOT MODEL
   XACRO FILES (FOR EXAMPLE, MODEL_BASE.XACRO AND MODEL_FORKLIFT.XACRO).
@@ -16,5 +16,4 @@
   Reference: package://ground_vehicle_kinematics/doc/kinematics_en.pdf
   - The chassis uses the RB-VOGUI DAE mesh for visual and the matching STL mesh for collision.
-  - The optional basket uses the RB-VOGUI std_basket mounting position.
   - Dynamics are intentionally simplified.
   Battery:
@@ -30,10 +29,9 @@
   <xacro:include filename="$(find robotics_description)/urdf/wheels/generic_macros/all_wheels_plugins.xacro"/>
   <xacro:include filename="$(find robotics_description)/urdf/gz_system_plugins/all_gz_system_plugins.xacro"/>
-  <xacro:include filename="$(find robotics_description)/urdf/extras/basket/basket_macros.xacro"/>
   <!-- ===================================================================== -->
   <!-- ARGS -->
   <!-- ===================================================================== -->
   <xacro:arg name="namespace"    default=""/>
-  <xacro:arg name="robot_name"   default="vog"/>
+  <xacro:arg name="robot_name"   default="rbvogui"/>
   <!--
   File containing the simulation configuration for the selected robot model.
@@ -45,6 +43,4 @@
   <xacro:arg name="body_use_collision"     default="True"/>
   <xacro:arg name="body_use_inertial"      default="True"/>
-  <xacro:arg name="use_basket_chassis"     default="True"/>
-  <xacro:arg name="use_basket_full"        default="False"/>
   <xacro:arg name="s_wheel_use_visual"     default="True"/>
   <xacro:arg name="s_wheel_use_v_mesh"     default="True"/>
@@ -86,15 +82,4 @@
   <xacro:property name="body_use_collision" value="$(arg body_use_collision)"/>
   <xacro:property name="body_use_inertial"  value="$(arg body_use_inertial)"/>
-  <xacro:property name="use_basket_chassis_raw" value="$(arg use_basket_chassis)"/>
-  <xacro:property name="use_basket_full_raw"    value="$(arg use_basket_full)"/>
-  <xacro:property name="use_basket_chassis"
-                  value="${str(use_basket_chassis_raw).strip().lower() in ('true', '1', 'yes')}"/>
-  <xacro:property name="use_basket_full"
-                  value="${str(use_basket_full_raw).strip().lower() in ('true', '1', 'yes')}"/>
-  <xacro:if value="${use_basket_chassis and use_basket_full}">
-    ${xacro.fatal(
-      "xacro args use_basket_chassis and use_basket_full cannot both be true"
-    )}
-  </xacro:if>
   <xacro:property name="top_body_size_x"        value="1.044"/>
   <xacro:property name="top_body_size_y"        value="0.650"/>
@@ -110,13 +95,10 @@
   <xacro:property name="chassis_joint_origin"   value="-0.012 0 0.1775 0 0 0"/>
   <xacro:property name="battery_joint_origin"   value="0.02952 0 0 0 0 0"/>
-  <xacro:property name="basket_joint_origin"    value="0.027732 0 0.2445 0 0 0"/>
   <xacro:property name="body_mesh_scale"        value="1.0 1.0 1.0"/>
-  <xacro:property name="chassis_visual_mesh"    value="robot_vog/meshes/rbvogui_chassis.dae"/>
-  <xacro:property name="chassis_collision_mesh" value="robot_vog/meshes/rbvogui_chassis.stl"/>
-  <xacro:property name="battery_mesh"           value="robot_vog/meshes/rbvogui_battery.stl"/>
+  <xacro:property name="chassis_visual_mesh"    value="robot_rbvogui_common/meshes/rbvogui_chassis.dae"/>
+  <xacro:property name="chassis_collision_mesh" value="robot_rbvogui_common/meshes/rbvogui_chassis.stl"/>
+  <xacro:property name="battery_mesh"           value="robot_rbvogui_common/meshes/rbvogui_battery.stl"/>
   <xacro:property name="battery_color"
                   value="${robot_prefix}battery_color 0.08235 0.08235 0.08235 1.0"/>
-  <xacro:property name="basket_color"
-                  value="${robot_prefix}basket_color 1.0 0.0 0.0 1.0"/>
   <xacro:property name="s_wheel_use_visual"   value="$(arg s_wheel_use_visual)"/>
   <xacro:property name="s_wheel_use_v_mesh"   value="$(arg s_wheel_use_v_mesh)"/>
@@ -274,20 +256,4 @@
     <xacro:origin_element origin="${battery_joint_origin}"/>
   </joint>
-  <!--
-  The basket mesh frame was moved to the center of its lower face. This offset preserves the old
-  RB-VOGUI std_basket visual position relative to chassis_link.
-  -->
-  <xacro:if value="${use_basket_chassis}">
-    <xacro:basket_chassis_macro prefix="${robot_prefix}"
-                                parent="${robot_prefix}chassis_link"
-                                joint_parent_fr_basket_fr="${basket_joint_origin}"
-                                color="${basket_color}"/>
-  </xacro:if>
-  <xacro:if value="${use_basket_full}">
-    <xacro:basket_full_macro prefix="${robot_prefix}"
-                             parent="${robot_prefix}chassis_link"
-                             joint_parent_fr_basket_fr="${basket_joint_origin}"
-                             basket_chassis_color="${basket_color}"/>
-  </xacro:if>
   <!--
   Definition of the steerable wheels.

File: urdf/model_base.xacro (robot description, xacro)
@@ -1,30 +1,20 @@
 <?xml version="1.0"?>
-<!--
-  This file publishes the `forklift` model of the `robot_vog` family.
-  The robot name inside the URDF stays `vog_forklift`.
-  This model extends the common VOG platform with the forklift module.
-  The forklift module contains:
-  - A simple fork.
-  - A realsense d435 camera (rgbd) mounted on the fork.
-  - A Robosense Airy lidar mounted on the back of the robot.
-  - A Robosense Airy lidar mounted on the front of the robot.
-  - A front bottom lidar mounted on the robot body.
--->
-<robot name="vog_forklift" xmlns:xacro="http://www.ros.org/wiki/xacro">
-  <!-- ===================================================================== -->
-  <!-- INCLUDES -->
-  <!-- ===================================================================== -->
-  <xacro:include filename="$(find robot_vog)/urdf/includes/common.xacro"/>
-  <xacro:include filename="$(find robot_vog)/urdf/includes/fork_simple_module.xacro"/>
+<robot name="rbvogui_base" xmlns:xacro="http://www.ros.org/wiki/xacro">
   <!--
-  The fork module creates the fork itself and the sensors mounted on it or above the body.
-  This model file only adds the Gazebo joint state publisher for the full assembled robot.
+  This file publishes the `base` model of the `robot_rbvogui_common` family.
+  The robot name inside the URDF stays `rbvogui_base`.
   -->
+  <xacro:include filename="$(find robot_rbvogui_common)/urdf/common.xacro"/>
+  <!-- A non-empty sim_file adds the simulation-only joint-state publisher. -->
   <xacro:if value="${sim_file != ''}">
     <gazebo>
+      <!--
+      Define a 'JointStatePublisher' Gazebo plugin to report the states of the joints.
+      -->
       <xacro:property name="joint_state_publisher_sim_cfg"
                       value="${sim_cfg.get('joint_state_publisher', dict())}"/>
       <xacro:if value="${joint_state_publisher_sim_cfg.get('enabled', False)}">
-        <xacro:property name="js_topic" value="${joint_state_publisher_sim_cfg.get('topic', '')}"/>
+        <xacro:property name="js_topic"
+                        value="${joint_state_publisher_sim_cfg.get('topic', '')}"/>
         <xacro:if value="${js_topic == ''}">
           ${xacro.fatal(
@@ -37,5 +27,4 @@
           <xacro:plugin_joint_state_publisher topic="${resolved_js_topic}">
             <joint_names>
-              <joint_name>${robot_prefix}${fork_name}_carriage_joint</joint_name>
               <joint_name>${robot_prefix}${front_left_wheel_name}_steering_joint</joint_name>
               <joint_name>${robot_prefix}${front_left_wheel_name}_rotation_joint</joint_name>

Commit message: feat: render models and bridge battery state
Split URDF rendering from model publishers and bridge the simulated battery state to ROS.

File: urdf/common.xacro (robot description, xacro)
@@ -2,7 +2,7 @@
 <robot name="rbvogui_common" xmlns:xacro="http://www.ros.org/wiki/xacro">
   <!--
-  Common xacro file for the RB-VOGUI robot with 4 steerable wheels.
-  THIS FILE IS NOT A COMPLETE ROBOT MODEL, IT IS MEANT TO BE INCLUDED IN THE SPECIFIC ROBOT MODEL
-  XACRO FILES (FOR EXAMPLE, MODEL_BASE.XACRO AND MODEL_FORKLIFT.XACRO).
+  Shared RB-VOGUI mobile-base Xacro for four steerable wheels.
+  This file is not a complete robot model. Entry-point Xacros such as model_base.xacro and
+  model_forklift.xacro include it, then add their own links, sensors, actuators, and Gazebo plugins.
   The base is composed of the RB-VOGUI chassis, battery and four steerable wheels:
   - Front-left wheel uses angle +alpha.
@@ -393,4 +393,51 @@
   <xacro:if value="${sim_file != ''}">
     <gazebo>
+      <xacro:property name="battery_sim_cfg" value="${sim_cfg.get('battery', dict())}"/>
+      <xacro:if value="${battery_sim_cfg.get('enabled', False)}">
+        <xacro:property name="battery_voltage" value="${battery_sim_cfg.get('voltage', '')}"/>
+        <xacro:property name="battery_capacity" value="${battery_sim_cfg.get('capacity', '')}"/>
+        <xacro:property name="battery_power_load" value="${battery_sim_cfg.get('power_load', '')}"/>
+        <xacro:if value="${battery_voltage == ''}">
+          ${xacro.fatal("battery.voltage is required when battery.enabled is true")}
+        </xacro:if>
+        <xacro:if value="${battery_capacity == ''}">
+          ${xacro.fatal("battery.capacity is required when battery.enabled is true")}
+        </xacro:if>
+        <xacro:if value="${battery_power_load == ''}">
+          ${xacro.fatal("battery.power_load is required when battery.enabled is true")}
+        </xacro:if>
+        <xacro:property name="battery_power_draining_topic"
+                        value="${battery_sim_cfg.get('power_draining_topic', '')}"/>
+        <xacro:if value="${battery_power_draining_topic != ''}">
+          <xacro:resolve_topic prop_id="battery_power_draining_topic"
+                               topic="${battery_power_draining_topic}"
+                               namespace="${robot_namespace}"/>
+        </xacro:if>
+        <xacro:property name="battery_stop_power_draining_topic"
+                        value="${battery_sim_cfg.get('stop_power_draining_topic', '')}"/>
+        <xacro:if value="${battery_stop_power_draining_topic != ''}">
+          <xacro:resolve_topic prop_id="battery_stop_power_draining_topic"
+                               topic="${battery_stop_power_draining_topic}"
+                               namespace="${robot_namespace}"/>
+        </xacro:if>
+        <xacro:plugin_linear_battery
+          name="main_battery"
+          voltage="${battery_voltage}"
+          capacity="${battery_capacity}"
+          power_load="${battery_power_load}"
+          fix_issue_225="${battery_sim_cfg.get('fix_issue_225', True)}"
+          open_circuit_voltage_constant_coef="${battery_sim_cfg.get('open_circuit_voltage_constant_coef', '')}"
+          open_circuit_voltage_linear_coef="${battery_sim_cfg.get('open_circuit_voltage_linear_coef', '')}"
+          initial_charge="${battery_sim_cfg.get('initial_charge', '')}"
+          resistance="${battery_sim_cfg.get('resistance', '')}"
+          smooth_current_tau="${battery_sim_cfg.get('smooth_current_tau', '')}"
+          invert_current_sign="${battery_sim_cfg.get('invert_current_sign', '')}"
+          start_draining="${battery_sim_cfg.get('start_draining', '')}"
+          power_draining_topic="${battery_power_draining_topic}"
+          stop_power_draining_topic="${battery_stop_power_draining_topic}"
+          enable_recharge="${battery_sim_cfg.get('enable_recharge', '')}"
+          charging_time="${battery_sim_cfg.get('charging_time', '')}"
+          recharge_by_topic="${battery_sim_cfg.get('recharge_by_topic', '')}"/>
+      </xacro:if>
       <!--
       To find the reference for the system Gazebo plugins:
